File: USB to Serial.brd (EAGLE design)
At the start: 72.1 x 83.8 mm, 44 parts, among them IC1 MEGA8-P, IC2 MEGA328-P, IC4 ATMega88*, Q1 16MHz, Q2 16MHz, Q3 16MHz, X1 PN61729-S

Commit message: finish
Parts:
- removed IC2: MEGA328-P, atmel:DIL28-3
- removed LED1: (no value), led:LED5MM
- added ZX1: 228-4817-00-0602J, con-3m:228-4817-00-0602J
- LED5, LED6: device led:LED3MM -> led:LED5MM
- R8: value 330 -> 10k; device adafruit:0207/7 -> rcl:0207/10
- R9: device adafruit:0207/7 -> rcl:0207/10
- moved LED2 42.6 mm to (73.7, 64.8)
- moved R9 37.0 mm to (55.9, 58.4), turned to 270 degrees
- moved LED5 27.9 mm to (57.1, 30.5)
- moved R8 20.4 mm to (16.5, 22.9), turned to 90 degrees
- moved R20 19.2 mm to (68.6, 14.0), turned to 180 degrees
- moved C8 18.5 mm to (78.7, 58.4)
- moved JP4 17.8 mm to (64.8, 24.1), turned to 270 degrees
- moved R17 17.3 mm to (68.6, 16.5), turned to 0 degrees
- moved R18 16.5 mm to (68.6, 19.1)
- moved R23 15.3 mm to (50.8, 17.8)
- moved LED6 15.2 mm to (52.1, 30.5)
- moved X3 14.0 mm to (67.3, 72.4)
- moved C9 13.7 mm to (73.7, 45.7), turned to 180 degrees
- moved IC4 12.7 mm to (64.8, 47.0)
- moved Q3 12.7 mm to (73.7, 53.3)
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Connections:
- removed net N$10: IC2.5
- removed net N$12: IC2.13, R8.2
- removed net N$15: LED1.A, R8.1
- removed net N$8: IC2.14, R9.2
- new net N$4: IC1.1, R8.2
- net DTR: now also X2.1, ZX1.1; no longer IC2.1
- net GND: now also X2.4, X3.6, ZX1.6; no longer IC2.22, LED1.K
- net MISO: now also X3.3, ZX1.18; no longer IC2.18
- net MOSI: now also X3.4, ZX1.17; no longer IC2.17
- net N$1: now also X3.5
- net N$9: now also ZX1.11; no longer IC2.11
- net OSC1: now also ZX1.9; no longer IC2.9
- net OSC2: now also ZX1.10; no longer IC2.10
- net RXD: now also X2.3, ZX1.3; no longer IC2.3
- net SCK: now also R9.2, X3.2, ZX1.19; no longer IC2.19
- net TXD: now also X2.2, ZX1.2; no longer IC2.2
- net VCC: now also R8.1, X3.1, ZX1.7; no longer IC2.20
Routing:
- net GND: track 388.3 -> 552.6 mm, vias 0 -> 2
- net VCC: track 184.6 -> 279.7 mm, vias 2 -> 6
- net MOSI: track 29.7 -> 102.5 mm
- net SCK: track 18.8 -> 91.5 mm
- net MISO: track 26.5 -> 96.6 mm
- net RXD: track 35.7 -> 82.1 mm
- net N$1: track 0.00 -> 39.7 mm, vias 0 -> 2
- net N$11: track 2.54 -> 38.7 mm, vias 0 -> 2
- net DTR: track 6.35 -> 29.6 mm
- net N$16: track 0.00 -> 18.8 mm
- net TXD: track 31.3 -> 49.8 mm
- net N$34: track 27.7 -> 45.5 mm
- net N$49: track 0.00 -> 15.9 mm
- net N$47: track 0.00 -> 15.8 mm
- net N$50: track 0.00 -> 11.2 mm
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Other:
- board size 72.1 x 83.8 mm -> 84.8 x 80 mm
- board text removed: "ANUNG"
