File: USB to Serial.sch (EAGLE design)
At the start: 44 parts, among them IC1 MEGA8-P, IC2 MEGA328-P, IC4 ATMega88*, Q1 16MHz, Q2 16MHz, Q3 16MHz, X1 PN61729-S

Commit message: finish
Parts:
- removed IC2: MEGA328-P, atmel:MEGA8-P
- removed LED1: (no value), led:LED5MM
- added ZX1: 228-4817-00-0602J, con-3m:228-4817-00-0602J
- LED5, LED6: device led:LED3MM -> led:LED5MM
- R8: value 330 -> 10k; device adafruit:R-US_0207/7 -> rcl:R-US_0207/10
- R9: device adafruit:R-US_0207/7 -> rcl:R-EU_0207/10
Connections:
- removed net N$10: IC2.PD3(INT1)
- removed net N$12: IC2.PD7(AIN1), R8.2
- removed net N$15: LED1.A, R8.1
- removed net N$8: IC2.PB0(ICP), R9.2
- new net N$4: IC1.PC6(/RESET), R8.2
- net DTR: now also X2-1.KL, ZX1.1; no longer IC2.PC6(/RESET)
- net GND: now also X2-4.KL, X3-6.KL, ZX1.6; no longer IC2.AGND, LED1.C
- net MISO: now also X3-3.KL, ZX1.18; no longer IC2.PB4(MISO)
- net MOSI: now also X3-4.KL, ZX1.17; no longer IC2.PB3(MOSI/OC2)
- net N$1: now also X3-5.KL
- net N$9: now also ZX1.11; no longer IC2.PD5(T1)
- net OSC1: now also ZX1.9; no longer IC2.PB6(XTAL1/TOSC1)
- net OSC2: now also ZX1.10; no longer IC2.PB7(XTAL2/TOSC2)
- net RXD: now also X2-3.KL, ZX1.3; no longer IC2.PD1(TXD)
- net SCK: now also R9.2, X3-2.KL, ZX1.19; no longer IC2.PB5(SCK)
- net TXD: now also X2-2.KL, ZX1.2; no longer IC2.PD0(RXD)
- net VCC: now also R8.1, X3-1.KL, ZX1.7; no longer IC2.AVCC
Other:
- moved on the sheet: LED2, R8
